File: pcb/hendrik/hendrik.sch (KiCad schematic (older format))
At the start: 42 parts, among them IC1 PIC32MK1024MCF064-I_PT, IC2 TPS54331DDAR, IC3 TC1262-3.3VDB, Q1 PN2222A, SW1 SW_Push, SW2 SW_Push

Commit message: PCB complete
Connections:
- net AD0 renamed GND
- net TX2 renamed RX1
Changed lines of the file:
@@
 TX1
 Text Label 10300 1700 0    50   ~ 0
-TX2
+RX1
 Text Label 16100 4850 0    50   ~ 0
 GND
@@
 INT1
 Text Label 16450 6150 0    50   ~ 0
-AD0
+GND
 $EndSCHEMATC
